File: Hardware/MicroViewUSB/MicroViewUSB.sch (EAGLE design)
At the start: 26 parts, among them J1 MICROVIEW-16ND, Q1 2N7002PW, U1 FT231XS

Commit message: Adding fids to both boards
Parts:
- added FID1, FID2: FIDUCIAL1X2, SparkFun-Aesthetics:FIDUCIAL1X2
Changed lines of the file:
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@@
 <part name="LOGO2" library="SparkFun-Aesthetics" deviceset="SFE_LOGO_FLAME" device=".1_INCH"/>
 <part name="LOGO3" library="SparkFun-Aesthetics" deviceset="SFE_LOGO_NAME_FLAME" device=".1_INCH"/>
+<part name="FID1" library="SparkFun-Aesthetics" deviceset="FIDUCIAL" device="1X2"/>
+<part name="FID2" library="SparkFun-Aesthetics" deviceset="FIDUCIAL" device="1X2"/>
 </parts>
 <sheets>
@@
 <instance part="LOGO2" gate="G$1" x="57.912" y="15.24"/>
 <instance part="LOGO3" gate="G$1" x="25.4" y="2.54"/>
+<instance part="FID1" gate="G$1" x="246.38" y="33.02"/>
+<instance part="FID2" gate="G$1" x="246.38" y="25.4"/>
 </instances>
 <busses>

Commit message: Staggering/increasing drill on headers
Also spacing out resistors, increasing header fp on MicroViewUSB.
Parts:
- renumbered J1 to J2
Changed lines of the file:
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@@
 <part name="C7" library="SparkFun-Capacitors" deviceset="0.1UF-25V(+80/-20%)(0603)" device="" value="0.1uF"/>
 <part name="U$2" library="SparkFun-Aesthetics" deviceset="5V" device=""/>
-<part name="J1" library="microView-temp" deviceset="MICROVIEW-16" device="ND"/>
 <part name="SUPPLY3" library="SparkFun-Aesthetics" deviceset="5V" device=""/>
 <part name="GND3" library="SparkFun-Aesthetics" deviceset="GND" device=""/>
@@
 <part name="FID1" library="SparkFun-Aesthetics" deviceset="FIDUCIAL" device="1X2"/>
 <part name="FID2" library="SparkFun-Aesthetics" deviceset="FIDUCIAL" device="1X2"/>
+<part name="J2" library="microView-temp" deviceset="MICROVIEW-16" device="ND"/>
 </parts>
 <sheets>
@@
 <instance part="C7" gate="G$1" x="99.06" y="76.2" rot="MR90"/>
 <instance part="U$2" gate="G$1" x="81.28" y="147.32"/>
-<instance part="J1" gate="G1" x="116.84" y="66.04"/>
 <instance part="SUPPLY3" gate="G$1" x="129.54" y="83.82"/>
 <instance part="GND3" gate="1" x="104.14" y="50.8"/>
@@
 <instance part="FID1" gate="G$1" x="246.38" y="33.02"/>
 <instance part="FID2" gate="G$1" x="246.38" y="25.4"/>
+<instance part="J2" gate="G1" x="116.84" y="66.04"/>
 </instances>
 <busses>
@@
 </segment>
 <segment>
-<pinref part="J1" gate="G1" pin="5V"/>
 <wire x1="127" y1="73.66" x2="129.54" y2="73.66" width="0.1524" layer="91"/>
 <wire x1="129.54" y1="73.66" x2="129.54" y2="83.82" width="0.1524" layer="91"/>
 <pinref part="SUPPLY3" gate="G$1" pin="5V"/>
+<pinref part="J2" gate="G1" pin="5V"/>
 </segment>
 </net>
@@
 </segment>
 <segment>
-<pinref part="J1" gate="G1" pin="GND"/>
 <pinref part="GND3" gate="1" pin="GND"/>
 <wire x1="106.68" y1="58.42" x2="104.14" y2="58.42" width="0.1524" layer="91"/>
 <wire x1="104.14" y1="58.42" x2="104.14" y2="53.34" width="0.1524" layer="91"/>
+<pinref part="J2" gate="G1" pin="GND"/>
 </segment>
 </net>
@@
 </segment>
 <segment>
-<pinref part="J1" gate="G1" pin="RXD"/>
 <wire x1="127" y1="58.42" x2="129.54" y2="58.42" width="0.1524" layer="91"/>
 <label x="129.54" y="58.42" size="1.27" layer="95" xref="yes"/>
+<pinref part="J2" gate="G1" pin="RXD"/>
 </segment>
 </net>
@@
 </segment>
 <segment>
-<pinref part="J1" gate="G1" pin="TXD"/>
 <wire x1="127" y1="60.96" x2="129.54" y2="60.96" width="0.1524" layer="91"/>
 <label x="129.54" y="60.96" size="1.27" layer="95" xref="yes"/>
+<pinref part="J2" gate="G1" pin="TXD"/>
 </segment>
 </net>
@@
 <segment>
 <pinref part="C7" gate="G$1" pin="1"/>
-<pinref part="J1" gate="G1" pin="RST"/>
 <wire x1="104.14" y1="76.2" x2="106.68" y2="76.2" width="0.1524" layer="91"/>
-</segment>
-</net>
+<pinref part="J2" gate="G1" pin="RST"/>
+</segment>
+</net>

Commit message: Updating r's and c's on USB board to prod. parts
Also rearranging some silk and traces.
Parts:
- removed LED1: Yellow, SparkFun-LED:LED1206
- removed LED2: Red, SparkFun-LED:LED1206
- removed LED3: Green, SparkFun-LED:LED1206
- removed R8, R9: 1k, SparkFun:RESISTOR0603-RES
- added D1: GREEN, SparkFun-LED:LED-GREENLARGE
- added D2: RED, SparkFun-LED:LED-RED1206
- added D3: Yellow, SparkFun-LED:LED-YELLOWLILYPAD
- added R4, R5: 1K, SparkFun-Resistors:1KOHM1/10W1%(0603)
- C1, C6: device SparkFun:CAP0603-CAP -> SparkFun-Capacitors:0.1UF-25V(+80/-20%)(0603)
- C4: value 0.1uF -> 10uF; device SparkFun:CAP0603-CAP -> SparkFun-Capacitors:10UF-16V-10%(TANT)
- C5: value 10uF -> 0.1uF; device SparkFun-Capacitors:CAP_POL1206 -> SparkFun-Capacitors:0.1UF-25V(+80/-20%)(0603)
- F1: device SparkFun:PTCSMD -> SparkFun-PowerIC:PTCSMD-W
- LOGO1: value OSHW-LOGOS -> SFE_LOGO_FLAME.1_INCH; device SparkFun-Aesthetics:OSHW-LOGOS -> SparkFun-Aesthetics:SFE_LOGO_FLAME.1_INCH
- LOGO2: value SFE_LOGO_FLAME.1_INCH -> OSHW-LOGOS; device SparkFun-Aesthetics:SFE_LOGO_FLAME.1_INCH -> SparkFun-Aesthetics:OSHW-LOGOS
- R1, R2: value 27 -> 10K; device SparkFun-Resistors:RESISTOR0603-RES -> SparkFun-Resistors:10KOHM1/10W1%(0603)0603
- R3: value 10k -> 1K; device SparkFun:RESISTOR0603-RES -> SparkFun-Resistors:1KOHM1/10W1%(0603)
- R6: value 10k -> 27; device SparkFun:RESISTOR0603-RES -> SparkFun-Resistors:RESISTOR0603-RES
- R7: value 1k -> 27; device SparkFun:RESISTOR0603-RES -> SparkFun-Resistors:RESISTOR0603-RES
- renumbered J2 to J1, JP2 to JP1
Connections:
- net 3.3V: now also R1.2; no longer R3.2
- net 5V: now also C4.+, C5.1, R2.2, R3.2, R4.2, R5.2; no longer C4.1, C5.+, R6.2, R7.1, R8.1, R9.1
- net D+: now also R7.1; no longer R2.1
- net D-: now also R6.1; no longer R1.1
- net DTR: now also C7.1, R2.1; no longer C7.2, R6.1
- net GND: now also C4.-, C5.2, D1.C; no longer C4.2, C5.-, LED3.C
- net N$1: now also D1.A, R5.1; no longer LED3.A, R9.2
- net N$10: now also D3.A, R3.1; no longer LED1.A, R7.2
- net N$12: now also R1.1; no longer R3.1
- net N$2: now also C7.2; no longer C7.1
- net N$6: now also R6.2; no longer R1.2
- net N$7: now also R7.2; no longer R2.2
- net N$8: now also D2.A, R4.1; no longer LED2.A, R8.2
- net RXLED: now also D3.C; no longer LED1.C
- net TXLED: now also D2.C; no longer LED2.C
Other:
- moved on the sheet: R1, R2, R3, R6, R7
